File: ConstantLoad.kicad_pcb (KiCad board)
At the start: 2 copper layers, 18 parts, among them P101 Battery Input, P102 CONN_01X03, P103 Current Sink Input, Q301 IRL640A, U201 LMV358, U401 AMS1117

Commit message: Add heatsink to PCB
Parts:
- added P301: Heatsink, Current:Heatsink_Aavid_6398BG, F.Cu at (137.2, 59.7)
- RV201, RV301: footprint Potentiometers:Potentiometer_Trimmer_Bourns_3006Y -> Potentiometers:Potentiometer_Triwood_RM-065
- moved P102 397.8 mm to (111.8, 53.3)
- moved U201 386.9 mm to (129.5, 72.4), turned to 180 degrees
- moved P101 385.2 mm to (111.8, 47.0)
- moved P103 385.1 mm to (111.8, 62.2)
- moved RV201 380.3 mm to (129.5, 92.7)
- moved D201 362.3 mm to (129.5, 82.5)
- moved R203 361.9 mm to (146.1, 88.9), turned to 270 degrees
- moved R202 358.2 mm to (156.2, 88.9), turned to 270 degrees
- moved RV301 357.0 mm to (113.0, 92.7)
- moved R201 351.7 mm to (151.1, 88.9), turned to 270 degrees
- moved U401 341.5 mm to (114.3, 76.2), turned to 180 degrees
- moved C401 340.9 mm to (121.9, 80.0), turned to 270 degrees
- moved C402 340.8 mm to (121.9, 74.9), turned to 270 degrees
- moved Q301 340.3 mm to (134.6, 63.5)
- moved R302 334.9 mm to (141.0, 88.9), turned to 270 degrees
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Other:
- board outline added: 50.8 x 50.8 mm

Commit message: Do pcb layout
Parts:
- P102: value CONN_01X03 -> Jumper
- R203: value R -> 27K
- R301: value R -> 68K
- RV201, RV301: value POT -> 10K
- U201: footprint Housings_SOIC:SOIC-8-1EP_3.9x4.9mm_Pitch1.27mm -> Housings_SOIC:SOIC-8_3.9x4.9mm_Pitch1.27mm
- U401: footprint TO_SOT_Packages_SMD:SOT-223 -> TO_SOT_Packages_SMD:SOT-223-3Lead_TabPin2
- moved C402 8.25 mm to (121.9, 83.2)
- moved C401 3.81 mm to (121.9, 76.2)
- moved P101 2.54 mm to (111.8, 49.5), turned to 180 degrees
Connections:
- C301 pad 1: +3V3 -> 3.3V
- C402 pad 1: +3V3 -> 3.3V
- R203 pad 1: Net-(R203-Pad1) -> 3.3V
- R203 pad 2: GND -> Net-(R203-Pad2)
- R301 pad 1: Net-(R301-Pad1) -> 3.3V
- R301 pad 2: GND -> Net-(R301-Pad2)
- RV201 pad 1: (no net) -> Net-(R203-Pad2)
- RV201 pad 2: +3V3 -> GND
- RV201 pad 3: Net-(R203-Pad1) -> (no net)
- RV301 pad 1: (no net) -> Net-(R301-Pad2)
- RV301 pad 2: +3V3 -> GND
- RV301 pad 3: Net-(R301-Pad1) -> (no net)
- U201 pad 3: Net-(R203-Pad1) -> Net-(R203-Pad2)
- U201 pad 5: Net-(R301-Pad1) -> Net-(R301-Pad2)
- U201 pad 8: +3V3 -> 3.3V
- U401 pad 1: /Power Regulation/Vin -> GND
- U401 pad 2: GND -> 3.3V
- U401 pad 3: (no net) -> /Power Regulation/Vin
Routing:
- net /Current Control/Current_Sink_In: track 0.00 -> 70.4 mm, vias 0 -> 1
- net 3.3V: track 0.00 -> 66.2 mm, vias 0 -> 5
- net Net-(R301-Pad2): track 0.00 -> 51.9 mm, vias 0 -> 2
- net Net-(R203-Pad2): track 0.00 -> 46.3 mm, vias 0 -> 1
- net Net-(R201-Pad2): track 0.00 -> 41.8 mm, vias 0 -> 2
- net Net-(Q301-Pad3): track 0.00 -> 37.2 mm, vias 0 -> 1
- net Net-(R302-Pad2): track 0.00 -> 27.3 mm, vias 0 -> 2
- net /Current Control/FET_Gate: track 0.00 -> 26.9 mm
- net /Power Regulation/Vin: track 0.00 -> 25.6 mm
- net Net-(D201-Pad1): track 0.00 -> 9.37 mm
- net GND: track 0.00 -> 5.42 mm, vias 0 -> 1
- net Net-(P101-Pad1): track 0.00 -> 3.81 mm
- added copper zone on B.Cu, net GND
- added copper zone on F.Cu, net GND
Other:
- net class Default: clearance 0.2 -> 0.254; trace_width 0.25 -> 0.254; via_dia 0.6 -> 0.889; via_drill 0.4 -> 0.635
- net class Power added: clearance 0.3048, trace_width 0.6096, via_dia 1.143, via_drill 0.762
- rule trace_clearance: 0.2 -> 0.254
- rule trace_min: 0.2 -> 0.254
- rule via_min_size: 0.4 -> 0.889

Commit message: Added logo
Parts:
- removed P301: Heatsink, Current:Heatsink_Aavid_6398BG
- added REF**: Heatsink_Aavid_6398BG, Current:Heatsink_Aavid_6398BG, F.Cu at (137.2, 59.7)
Changed lines of the file:
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@@
   (page A4)
   (layers
-    (0 F.Cu signal hide)
+    (0 F.Cu signal)
     (31 B.Cu signal)
     (32 B.Adhes user)
@@
     )
   )
-  (module Current:Heatsink_Aavid_6398BG (layer F.Cu)
-    (at 137.16 59.69)
-    (fp_text reference P301 (at 5.588 -2.286) (layer F.SilkS)
-      (effects (font (size 1 1) (thickness 0.15)))
-    )
-    (fp_text value Heatsink (at -0.254 -2.286) (layer F.Fab)
-      (effects (font (size 1 1) (thickness 0.15)))
-    )
-    (fp_line (start -12.7 1.524) (end -12.7 12.7) (layer F.SilkS) (width 0.15))
-    (fp_line (start -12.7 12.7) (end -20.955 12.7) (layer F.SilkS) (width 0.15))
-    (fp_line (start -20.955 12.7) (end -20.955 -12.7) (layer F.SilkS) (width 0.15))
-    (fp_line (start -20.955 -12.7) (end 20.955 -12.7) (layer F.SilkS) (width 0.15))
-    (fp_line (start 11.43 0.7874) (end -11.3792 0.7874) (layer F.SilkS) (width 0.15))
-    (fp_line (start 20.955 -12.7) (end 20.955 12.7) (layer F.SilkS) (width 0.15))
-    (fp_line (start 20.955 12.7) (end 12.7 12.7) (layer F.SilkS) (width 0.15))
-    (fp_line (start 12.7 12.7) (end 12.7 1.905) (layer F.SilkS) (width 0.15))
-    (pad "" np_thru_hole circle (at 12.7 0) (size 2.8956 2.8956) (drill 2.8956) (layers *.Cu *.Mask))
-    (pad "" np_thru_hole circle (at -12.7 0) (size 2.8956 2.8956) (drill 2.8956) (layers *.Cu *.Mask))
-  )
   (module Housings_SOIC:SOIC-8_3.9x4.9mm_Pitch1.27mm (layer F.Cu)
     (at 129.54 72.39 180)
@@
     )
   )
+  (module Current:Heatsink_Aavid_6398BG (layer F.Cu)
+    (at 137.16 59.69)
+    (fp_text reference REF** (at 16.891 14.859) (layer F.SilkS)
+      (effects (font (size 1 1) (thickness 0.15)))
+    )
+    (fp_text value Heatsink_Aavid_6398BG (at -0.254 -2.286) (layer F.Fab)
+      (effects (font (size 1 1) (thickness 0.15)))
+    )
+    (fp_line (start -12.7 1.524) (end -12.7 12.7) (layer F.SilkS) (width 0.15))
+    (fp_line (start -12.7 12.7) (end -20.955 12.7) (layer F.SilkS) (width 0.15))
+    (fp_line (start -20.955 12.7) (end -20.955 -12.7) (layer F.SilkS) (width 0.15))
+    (fp_line (start -20.955 -12.7) (end 20.955 -12.7) (layer F.SilkS) (width 0.15))
+    (fp_line (start 11.43 0.7874) (end -11.3792 0.7874) (layer F.SilkS) (width 0.15))
+    (fp_line (start 20.955 -12.7) (end 20.955 12.7) (layer F.SilkS) (width 0.15))
+    (fp_line (start 20.955 12.7) (end 12.7 12.7) (layer F.SilkS) (width 0.15))
+    (fp_line (start 12.7 12.7) (end 12.7 1.905) (layer F.SilkS) (width 0.15))
+    (pad 2 thru_hole circle (at 12.7 0) (size 3.556 3.556) (drill 2.8956) (layers *.Cu *.Mask))
+    (pad 1 thru_hole circle (at -12.7 0) (size 3.556 3.556) (drill 2.8956) (layers *.Cu *.Mask))
+  )
   (gr_line (start 160.02 44.45) (end 109.22 44.45) (angle 90) (layer Edge.Cuts) (width 0.15))

Commit message: Generate Gerbers
Parts:
- added REF***: OSHW-Logo2_9.8x8mm_SilkScreen, Symbols:OSHW-Logo2_9.8x8mm_SilkScreen, B.Cu at (137.3, 52.2)
